File: kicad/usb_thermo_logger/usb_thermo_logger.sch (KiCad schematic (older format))
At the start: 50 parts, among them J1 690-005-299-043, J2 SWD, J3 RESET, J4 BOOT0, U1 STM32F070CBT6, U2 24AA02-OT, U3 MAX31855KASA, U4 MAX31855KASA, U5 PCA9531, U6 LD3985M33R_SOT23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

Commit message: LED display changes, added OpenSCAD
Parts:
- removed U5: PCA9531, Package_SO:SOIC-16_3.9x9.9mm_P1.27mm, symbol thermologger:PCA9531
- added C21: 100n, Capacitor_SMD:C_0603_1608Metric, symbol Device:C
- added U5: SN74LVC06ADR, Package_SO:SOIC-14_3.9x8.7mm_P1.27mm, symbol 74xx:74LS06
- D2, D3: footprint LED_THT:LED_D5.0mm-4_RGB -> LED_SMD:LED_Avago_PLCC4_3.2x2.8mm_CW
- R3, R6: value 560R -> 1k
- R4, R5, R7, R8: value 560R -> 2k2
Connections:
- net labels added: BLUE1, BLUE2, GREEN1, GREEN2, RED1, RED2
- wire segments 224 -> 222
Other:
- moved on the sheet: C10, C11, C12, C9, D3, FB5, R6, R7, U6

Commit message: Layout changes
Parts:
- removed R1: 100k, Resistor_SMD:R_0603_1608Metric, symbol Device:R
- added TP1: SCL, TestPoint:TestPoint_Pad_1.0x1.0mm, symbol Connector:TestPoint
- added TP10: DM, TestPoint:TestPoint_Pad_1.0x1.0mm, symbol Connector:TestPoint
- added TP11: DP, TestPoint:TestPoint_Pad_1.0x1.0mm, symbol Connector:TestPoint
- added TP2: SDA, TestPoint:TestPoint_Pad_1.0x1.0mm, symbol Connector:TestPoint
- added TP3: VCC, TestPoint:TestPoint_Pad_1.0x1.0mm, symbol Connector:TestPoint
- added TP4: GND, TestPoint:TestPoint_Pad_1.0x1.0mm, symbol Connector:TestPoint
- added TP5: CS1, TestPoint:TestPoint_Pad_1.0x1.0mm, symbol Connector:TestPoint
- added TP6: SCK, TestPoint:TestPoint_Pad_1.0x1.0mm, symbol Connector:TestPoint
- added TP7: MISO, TestPoint:TestPoint_Pad_1.0x1.0mm, symbol Connector:TestPoint
- added TP8: VIN, TestPoint:TestPoint_Pad_1.0x1.0mm, symbol Connector:TestPoint
- added TP9: CS2, TestPoint:TestPoint_Pad_1.0x1.0mm, symbol Connector:TestPoint
- U3, U4: symbol Sensor_Temperature:MAX31855KASA -> usb_thermo_logger-rescue:MAX31855KASA-Sensor_Temperature
- U7: symbol Power_Protection:USBLC6-2SC6 -> usb_thermo_logger-rescue:USBLC6-2SC6-Power_Protection
Connections:
- net labels removed: ID
- wire segments 222 -> 238
Other:
- moved on the sheet: C2, C4, XTAL2
